File: ACBoard.kicad_pcb (KiCad board)
At the start: 2 copper layers, 61.6 x 55.2 mm, 32 parts, among them J1 Conn_02x20_Odd_Even, J2 Conn_02x20_Odd_Even, J3 Conn_01x02_Male, J4 Conn_01x02_Female, J5 Conn_01x02_Female, T1 CSE185L, U1 TLP561, U2 TLP561, U3 ADS7822U

Commit message: data19
Parts:
- removed C1: 10u, Capacitor_SMD:C_0805_2012Metric_Pad1.18x1.45mm_HandSolder
- removed C2: 0.1u, Capacitor_SMD:C_1206_3216Metric_Pad1.33x1.80mm_HandSolder
- removed D1, D2: Q_TRIAC_A1A2G, Package_TO_SOT_THT:TO-220-3_Horizontal_TabDown
- removed D3: VS3V3BC1EST15R, Diode_SMD:D_0201_0603Metric_Pad0.64x0.40mm_HandSolder
- removed D4, D5: D, Diode_THT:D_5W_P12.70mm_Horizontal
- removed DH1, DH2, DH3, DH4, DH5: Drill, locallib:Drill
- removed H1, H2: heatsink, locallib:heatsink
- removed J1: Conn_02x20_Odd_Even, Connector_PinSocket_2.54mm:PinSocket_2x20_P2.54mm_Vertical
- removed J2: Conn_02x20_Odd_Even, Connector_PinHeader_2.54mm:PinHeader_2x20_P2.54mm_Vertical
- removed J3: Conn_01x02_Male, locallib:ACinlet
- removed J4, J5: Conn_01x02_Female, locallib:AcOutlet
- removed R1, R2, R3, R4: 100, Resistor_SMD:R_0603_1608Metric_Pad0.98x0.95mm_HandSolder
- removed R5: 67, Resistor_SMD:R_0603_1608Metric_Pad0.98x0.95mm_HandSolder
- removed R6, R7: 1k, Resistor_SMD:R_0603_1608Metric_Pad0.98x0.95mm_HandSolder
- removed RV1, RV2: Varistor, Varistor:RV_Disc_D9mm_W3.8mm_P5mm
- removed T1: CSE185L, locallib:XFMR_CSE185L
- removed U1, U2: TLP561, Package_DIP:DIP-5-6_W7.62mm
- removed U3: ADS7822U, locallib:SOIC127P599X175-8N
Routing:
- net GND: track 224.4 -> 0.00 mm, vias 114 -> 0
- net +3V3: track 128.6 -> 0.00 mm
- net /GPIO17: track 83.1 -> 0.00 mm
- net /GPIO27: track 72.7 -> 0.00 mm
- net Net-(D3-Pad2): track 72.5 -> 0.00 mm
- net /GPIO10: track 72.2 -> 0.00 mm
- net /GPIO11: track 67.3 -> 0.00 mm, vias 1 -> 0
- net /FS: track 64.2 -> 0.00 mm
- net /GPIO9: track 63.8 -> 0.00 mm, vias 1 -> 0
- net /GPIO26: track 62.5 -> 0.00 mm
- net VAC: track 61.1 -> 0.00 mm
- net /GPIO5: track 60.9 -> 0.00 mm
- net Net-(C1-Pad1): track 59.7 -> 0.00 mm
- net /USB_DM: track 59.7 -> 0.00 mm
- net /EEPROM_SDA: track 59.6 -> 0.00 mm
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- removed copper zone on B.Cu, net GND
- removed copper zone on F.Cu, net GND
Other:
- board outline removed
