File: ACBoard.kicad_sch (KiCad schematic)
At the start: 25 parts, among them J1 Conn_02x20_Odd_Even, J2 Conn_02x20_Odd_Even, J3 Conn_01x02_Male, J4 Conn_01x02_Female, J5 Conn_01x02_Female, T1 CSE185L, U1 TLP561, U2 TLP561, U3 ADS7822U

Commit message: Update ACBoard.kicad_sch
Parts:
- R5: footprint Resistor_SMD:R_0603_1608Metric_Pad0.98x0.95mm_HandSolder -> Resistor_SMD:R_2010_5025Metric_Pad1.40x2.65mm_HandSolder
Changed lines of the file:
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@@
       (effects (font (size 1.27 1.27)) (justify left))
     )
-    (property "Footprint" "Resistor_SMD:R_0603_1608Metric_Pad0.98x0.95mm_HandSolder" (id 2) (at 202.692 63.5 90)
+    (property "Footprint" "Resistor_SMD:R_2010_5025Metric_Pad1.40x2.65mm_HandSolder" (id 2) (at 202.692 63.5 90)
       (effects (font (size 1.27 1.27)) hide)
     )
@@
     )
     (path "/0d402606-3120-4980-8456-8f91cb64a988"
-      (reference "R5") (unit 1) (value "67") (footprint "Resistor_SMD:R_0603_1608Metric_Pad0.98x0.95mm_HandSolder")
+      (reference "R5") (unit 1) (value "67") (footprint "Resistor_SMD:R_2010_5025Metric_Pad1.40x2.65mm_HandSolder")
     )
     (path "/fe4fefbf-4e6d-41f6-b3b2-a9a978e16f7d"

Commit message: data19
Parts:
- removed C1: 10u, Capacitor_SMD:C_0805_2012Metric_Pad1.18x1.45mm_HandSolder, symbol Device:C
- removed C2: 0.1u, Capacitor_SMD:C_1206_3216Metric_Pad1.33x1.80mm_HandSolder, symbol Device:C
- removed D1, D2: Q_TRIAC_A1A2G, Package_TO_SOT_THT:TO-220-3_Horizontal_TabDown, symbol Device:Q_TRIAC_A1A2G
- removed D3: VS3V3BC1EST15R, Diode_SMD:D_0201_0603Metric_Pad0.64x0.40mm_HandSolder, symbol Device:D_TVS
- removed D4, D5: D, Diode_THT:D_5W_P12.70mm_Horizontal, symbol Device:D
- removed J3: Conn_01x02_Male, locallib:ACinlet, symbol Connector:Conn_01x02_Male
- removed J4, J5: Conn_01x02_Female, locallib:AcOutlet, symbol Connector:Conn_01x02_Female
- removed R1, R2, R3, R4: 100, Resistor_SMD:R_0603_1608Metric_Pad0.98x0.95mm_HandSolder, symbol Device:R
- removed R5: 67, Resistor_SMD:R_2010_5025Metric_Pad1.40x2.65mm_HandSolder, symbol Device:R
- removed R6, R7: 1k, Resistor_SMD:R_0603_1608Metric_Pad0.98x0.95mm_HandSolder, symbol Device:R
- removed RV1, RV2: Varistor, Varistor:RV_Disc_D9mm_W3.8mm_P5mm, symbol Device:Varistor
- removed T1: CSE185L, locallib:XFMR_CSE185L, symbol locallib:CSE185L
- removed U1, U2: TLP561, Package_DIP:DIP-5-6_W7.62mm, symbol locallib:TLP561
- removed U3: ADS7822U, locallib:SOIC127P599X175-8N, symbol locallib:ADS7822U
- added AE?: Antenna, symbol Device:Antenna
- added C? (x4): C, symbol Device:C
- added D?: LED, symbol Device:LED
- added JP? (x3): SolderJumper_2_Open, symbol Jumper:SolderJumper_2_Open
- added R? (x6): R, symbol Device:R
- added U?: Si4831, symbol locallib:Si4831
- added Y?: Crystal, symbol Device:Crystal
Connections:
- net +3V3: now also C?.2, R?.1, R?.1, R?.2, U?.20 (VDD1), U?.21 (VDD2)
- net GND: now also C?.1, R?.2, U?.13 (GND), U?.14 (GND), U?.9 (RFGND)
- new net: JP?.2 (B), R?.1, R?.2 (x3)
- new net: C?.2, R?.2, U?.15 (*RST)
- new net: AE?.1 (A), U?.8 (FMI)
- new net: C?.1, U?.22 (DBYP)
- new net: C?.1, U?.18 (Xtalo), Y?.1
- new net: C?.2, C?.2
- new net: C?.1, U?.19 (Xtali), Y?.2
- new net: JP?.1 (A), JP?.1 (A), JP?.1 (A), U?.5 (Band)
- new net: D?.2 (A), R?.1
- new net LAN_EN: D?.1 (K), U?.1 (Stereo)
- new net Lout: U?.24 (Lout)
- new net Rout: U?.23 (Rout)
- no-connect marks 0 -> 5

Commit message: dara2
Parts:
- removed AE?: Antenna, symbol Device:Antenna
- removed C? (x4): C, symbol Device:C
- removed D?: LED, symbol Device:LED
- removed JP? (x3): SolderJumper_2_Open, symbol Jumper:SolderJumper_2_Open
- removed R? (x6): R, symbol Device:R
- removed U?: Si4831, symbol locallib:Si4831
- removed Y?: Crystal, symbol Device:Crystal
- added AE?: Antenna, symbol Device:Antenna
- added C? (x4): C, symbol Device:C
- added JP?: SolderJumper_2_Open, symbol Jumper:SolderJumper_2_Open
- added L?: L, symbol Device:L
- added R? (x4): R, symbol Device:R
- added U?: Si4832, symbol locallib:Si4832
Connections:
- net +3V3: now also C?.1, R?.1, R?.2, R?.2, U?.14 (VDD)
- net DIN: now also U?.16 (Rout)
- net FS: now also U?.1 (Lout)
- net GND: now also C?.2, C?.2, C?.2, JP?.1 (A), R?.2, U?.15 (GND), U?.7 (RfGnd)
- net GPIO18: now also U?.2 (Dclk)
- net GPIO2: now also U?.12 (SDIO)
- net GPIO27: now also C?.1, R?.2, U?.9 (*Rst)
- net GPIO3: now also U?.11 (SCLK)
- net GPIO4: now also U?.13 (RCLK)
- new net: R?.1, U?.3 (IntB)
- new net: R?.1, U?.4 (IO1)
- new net: AE?.1 (A), L?.2, U?.6 (FMI)
- new net: C?.2, U?.8 (AMI)
- new net: C?.1, L?.1
- new net SenB: C?.1, JP?.2 (B), R?.1, U?.10 (SenB)
- no-connect marks 5 -> 1
Other:
- note added: "https://gist.github.com/JonathanThorpe/f23480c781ca62a28647"

Commit message: data10
Parts:
- added C?: C, symbol Device:C
- added JP?: SolderJumper_2_Open, symbol Jumper:SolderJumper_2_Open
- added R? (x3): R, symbol Device:R
- added U?: PCM5122PW, Package_SO:TSSOP-28_4.4x9.7mm_P0.65mm, symbol Audio:PCM5122PW
- U?: value Si4832 -> Si4732
Connections:
- net +3V3: now also R?.2, R?.2, U?.1 (CPVDD), U?.28 (DVDD), U?.8 (AVDD)
- net DOUT: now also U?.22 (DIN)
- net FS: now also U?.23 (LRCK)
- net GND: now also C?.2, JP?.1 (A), R?.1
- net GPIO18: now also U?.21 (BCK)
- net GPIO2: now also U?.11 (SDA/MOSI/ATT2)
- net GPIO3: now also U?.12 (SCL/MC/ATT1)
- new net: C?.1, JP?.2 (B), R?.1
- new net: R?.2, U?.17 (MODE1)
- new net: R?.1, U?.18 (MODE2/MS)
- new net Adr1: U?.24 (ADR1/MISO/FMT)

Commit message: Anotaiton
Parts:
- added C10, C14, C16, C17, C19, C3, C4, C8, C9: C, symbol Device:C
- added C13, C15, C18, C6, C7: C_Polarized, symbol Device:C_Polarized
- added D1, D2: LED, symbol Device:LED
- added J3: SJ1-3523N, CUI_SJ1-3523N, symbol locallib:SJ1-3523N
- added JP3: SolderJumper_2_Open, symbol Jumper:SolderJumper_2_Open
- added R10, R13, R2, R5, R6, R9: R, symbol Device:R
- gave numbers to parts that had none: 18
Connections:
- net GPIO22' is gone; now on net GPIO22: J2.15 (Pin_15)
- net +3V3: now also C13.1, C14.1, C15.1, C16.1, C18.1, C19.1, R10.2, R13.2, R9.2
- net Adr1: now also C12.1, JP2.2 (B), R12.1
- net GND: now also U1.27 (DGND), U1.3 (CPGND), U1.9 (AGND), C10.2, C13.2, C14.2, C15.2, C16.2, C17.2, C18.2, C19.2, C3.2, C6.2, C7.2, C8.2, C9.2, J3.1, JP3.1 (A), R2.1
- net GPIO27': now also U1.13 (GPIO5/ATT0)
- net GPIO4: no longer J2.7 (Pin_7)
- net at U1.10 (VCOM/DEMP): now also C7.1
- net IODAC4: now reaches U1.14 (GPIO4/MAST)
- net IODAC4: now also D2.2 (A)
- net IODAC3: now reaches U1.15 (GPIO3/AGNS)
- net IODAC3: now also D1.2 (A)
- net Adr2: now reaches U1.16 (ADR2/GPIO2/DOUT)
- net Adr2: now also C17.1, JP3.2 (B), R13.1
- net GPIO4': now reaches U1.19 (GPIO6/FLT)
- net GPIO4': now also J2.7 (Pin_7)
- net at U1.2 (CAPP): now also C4.1
- net at U1.20 (SCK): now also R2.2
- net at U1.26 (LDOO): now also C6.1, C9.1
- net at U1.4 (CAPM): now also C4.2
- net at U1.5 (VNEG): now also C3.1
- net at U1.6 (OUTL): now also R5.1
- net at U1.7 (OUTR): now also R6.2
- new net: C8.1, J3.2, R6.1
- new net: C10.1, J3.3, R5.2
- new net: D2.1 (K), R10.1
- new net: D1.1 (K), R9.1
Other:
- moved on the sheet: C12, JP2, R12

Commit message: l
Parts:
- added R?: R, symbol Device:R
Connections:
- net +3V3: now also R?.1
- net at U1.25 (XSMT): now also R?.2
Other:
- note added: "https://nabe.adiary.jp/0566"
Changed lines of the file:
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@@
+    (stroke (width 0) (type default) (color 0 0 0 0))
+  )
+  (wire (pts (xy 110.49 151.13) (xy 114.3 151.13))
     (stroke (width 0) (type default) (color 0 0 0 0))
   )
@@
   (text "https://gist.github.com/JonathanThorpe/f23480c781ca62a28647"
     (at 212.09 86.36 0)
+    (effects (font (size 1.27 1.27)) (justify left bottom))
+  )
+  (text "https://nabe.adiary.jp/0566" (at 31.75 149.86 0)
+    (effects (font (size 1.27 1.27)) (justify left bottom))
+  )
+  (text "https://gist.github.com/JonathanThorpe/f23480c781ca62a28647"
+    (at 33.02 153.67 0)
     (effects (font (size 1.27 1.27)) (justify left bottom))
   )
@@
     (pin "1")
     (pin "2")
+  )
+  (symbol (lib_id "power:+3V3") (at 110.49 151.13 0) (unit 1)
+    (in_bom yes) (on_board yes)
+    (property "Reference" "#PWR?" (id 0) (at 110.49 154.94 0)
+      (effects (font (size 1.27 1.27)) hide)
+    )
+    (property "Value" "+3V3" (id 1) (at 110.871 146.7358 0))
+    (property "Footprint" "" (id 2) (at 110.49 151.13 0)
+      (effects (font (size 1.27 1.27)) hide)
+    )
+    (property "Datasheet" "" (id 3) (at 110.49 151.13 0)
+      (effects (font (size 1.27 1.27)) hide)
+    )
+    (pin "1")
   )
   (symbol (lib_id "power:GND") (at 214.63 146.05 0) (unit 1)
@@
     (pin "1")
   )
+  (symbol (lib_id "Device:R") (at 114.3 147.32 180) (unit 1)
+    (in_bom yes) (on_board yes) (fields_autoplaced)
+    (property "Reference" "R?" (id 0) (at 116.078 146.4853 0)
+      (effects (font (size 1.27 1.27)) (justify right))
+    )
+    (property "Value" "R" (id 1) (at 116.078 149.0222 0)
+      (effects (font (size 1.27 1.27)) (justify right))
+    )
+    (property "Footprint" "" (id 2) (at 116.078 147.32 90)
+      (effects (font (size 1.27 1.27)) hide)
+    )
+    (property "Datasheet" "~" (id 3) (at 114.3 147.32 0)
+      (effects (font (size 1.27 1.27)) hide)
+    )
+    (pin "1")
+    (pin "2")
+  )
   (symbol (lib_id "power:+3V3") (at 142.24 72.39 0) (unit 1)
     (in_bom yes) (on_board yes)
@@
       (reference "#PWR0122") (unit 1) (value "GND") (footprint "")
     )
+    (path "/111a9cf1-58cb-4410-953d-499d23c85f0f"
+      (reference "#PWR?") (unit 1) (value "+3V3") (footprint "")
+    )
     (path "/dd4b4fed-ba41-492c-9965-870ff0044781"
       (reference "AE1") (unit 1) (value "Antenna") (footprint "")
@@
       (reference "R13") (unit 1) (value "R") (footprint "")
     )
+    (path "/d31f952d-21f4-46fe-988d-d75bf089ad89"
+      (reference "R?") (unit 1) (value "R") (footprint "")
+    )
     (path "/bad15ef1-4174-4239-b07e-7b1abace56d9"
