File: ACBoard.kicad_sch (KiCad schematic)
At the start: 49 parts, among them J1 Conn_02x20_Odd_Even, J2 Conn_02x20_Odd_Even, J3 SJ1-3523N, U1 PCM5122PW, U2 Si4732, U3 CM1213A-02

Commit message: data
Parts:
- removed R2: R, symbol Device:R
- added C? (x2): C, symbol Device:C
- added C? (x2): C_Polarized, symbol Device:C_Polarized
- added J? (x2): Conn_Coaxial, symbol Connector:Conn_Coaxial
- added SW?: SW_SPDT, symbol Switch:SW_SPDT
- added U?: AP2120N-3.3TRG1, Package_TO_SOT_SMD:SOT-23, symbol Regulator_Linear:AP2127N-2.5
- added X?: DSC6001JI2A-022.5792, symbol Oscillator:SG-210STF
- added X?: SIT8008BI-23-33E-24.576000, symbol Oscillator:SG-210STF
Connections:
- net +3V3: now also X?.4 (Vcc), X?.4 (Vcc); no longer U1.1 (CPVDD), U1.8 (AVDD)
- net +5V: now also C?.1, C?.1, U?.3 (VI)
- net GND: now also C?.2, C?.2, C?.2, C?.2, J?.2 (Ext), J?.2 (Ext), U?.1 (GND), X?.2 (GND), X?.2 (GND)
- net GPIO27': no longer U1.13 (GPIO5/ATT0)
- net GPIO4': no longer U1.19 (GPIO6/FLT)
- net OUTR: now reaches C8.1, R6.1
- net OUTR: now also J3.3, J?.1 (In); no longer J3.2
- net OUTL: now reaches C10.1, R5.2
- net OUTL: now also J3.2, J?.1 (In); no longer J3.3
- net at C1.1, C?.2, U3.3 (CH2): now also SW?.2 (B); no longer AE2.2, C?.1, L1.1
- net SCKDAC: now reaches U1.20 (SCK)
- net SCKDAC: now also X?.3 (OUT), X?.3 (OUT)
- net IODAC3 renamed DACIO3
- net DACIO3: now also X?.1 (~{ST})
- net IODAC4 renamed DACIO5
- net DACIO5: now also U1.13 (GPIO5/ATT0)
- new net: AE2.2, C?.1, SW?.1 (A)
- new net: L1.1, SW?.3 (C)
- new net +3.3VA: C?.1, C?.1, U1.1 (CPVDD), U1.8 (AVDD), U?.2 (VO)
- new net DACIO6: U1.19 (GPIO6/FLT), X?.1 (~{ST})
Other:
- moved on the sheet: AE2, C?, L1

Commit message: data
Parts:
- added C26: 47u, symbol Device:C_Polarized
- C10, C8: value C -> 2.2n
- C11, C12, C14, C16, C17, C19, C2, C5, C9: value C -> 0.1u
- C13, C15, C18, C6, C7: value C_Polarized -> 10u
- C21: renamed from C?; value C -> 10nH
- C22, C25: renamed from C?; value C_Polarized -> 10u
- C23, C24: renamed from C?; value C -> 2.2u
- C3, C4: value C -> 2.2u
- J3: footprint CUI_SJ1-3523N -> locallib:CUI_SJ1-3523N
- J4, J5: renamed from J?; value Conn_Coaxial -> RCA
- L2: renamed from L?; value L -> 100nH
- R1, R11, R12, R13, R3, R4, R7, R8: value R -> 10k
- R10, R5, R6: value R -> 470
- R2: renamed from R?; value R -> 10k
- X1, X2: renamed from X?; footprint (none) -> Oscillator:Oscillator_SMD_SeikoEpson_SG8002LB-4Pin_5.0x3.2mm; symbol Oscillator:SG-210STF -> Oscillator:SG-5032CCN
- gave numbers to parts that had none: 3
Connections:
- net +3.3VA: now also C26.1
- net GND: now also C26.2

Commit message: d
Parts:
- AE1: footprint (none) -> Connector_PinHeader_2.54mm:PinHeader_1x01_P2.54mm_Vertical
- AE2: footprint (none) -> Connector_PinHeader_2.54mm:PinHeader_1x02_P2.54mm_Vertical
- C1: footprint (none) -> Capacitor_SMD:C_1206_3216Metric_Pad1.33x1.80mm_HandSolder
Changed lines of the file:
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@@
       (effects (font (size 1.27 1.27)) (justify left))
     )
-    (property "Footprint" "" (id 2) (at 134.62 29.21 0)
+    (property "Footprint" "Connector_PinHeader_2.54mm:PinHeader_1x01_P2.54mm_Vertical" (id 2) (at 134.62 29.21 0)
       (effects (font (size 1.27 1.27)) hide)
     )
@@
     (property "Reference" "C1" (id 0) (at 146.05 38.5912 90))
     (property "Value" "0.47u" (id 1) (at 146.05 41.1281 90))
-    (property "Footprint" "" (id 2) (at 149.86 43.4848 0)
+    (property "Footprint" "Capacitor_SMD:C_1206_3216Metric_Pad1.33x1.80mm_HandSolder" (id 2) (at 149.86 43.4848 0)
       (effects (font (size 1.27 1.27)) hide)
     )
@@
     (property "Reference" "AE2" (id 0) (at 107.95 38.2102 90))
     (property "Value" "Antenna_Loop" (id 1) (at 107.95 40.7471 90))
-    (property "Footprint" "" (id 2) (at 107.95 46.99 0)
+    (property "Footprint" "Connector_PinHeader_2.54mm:PinHeader_1x02_P2.54mm_Vertical" (id 2) (at 107.95 46.99 0)
       (effects (font (size 1.27 1.27)) hide)
     )
@@
     )
     (path "/dd4b4fed-ba41-492c-9965-870ff0044781"
-      (reference "AE1") (unit 1) (value "Antenna") (footprint "")
+      (reference "AE1") (unit 1) (value "Antenna") (footprint "Connector_PinHeader_2.54mm:PinHeader_1x01_P2.54mm_Vertical")
     )
     (path "/f5661775-35d9-4814-b6c8-86faf7af6737"
-      (reference "AE2") (unit 1) (value "Antenna_Loop") (footprint "")
+      (reference "AE2") (unit 1) (value "Antenna_Loop") (footprint "Connector_PinHeader_2.54mm:PinHeader_1x02_P2.54mm_Vertical")
     )
     (path "/ebf31f48-a45e-406a-9303-f1b18920d1b8"
-      (reference "C1") (unit 1) (value "0.47u") (footprint "")
+      (reference "C1") (unit 1) (value "0.47u") (footprint "Capacitor_SMD:C_1206_3216Metric_Pad1.33x1.80mm_HandSolder")
     )
     (path "/86ddee13-68ce-4a53-8769-536e010c73d8"

Commit message: da
Other:
- note added: "https://github.com/raspberrypi/linux/blob/rpi-5.15.y/sound/soc/bcm/hifiberry_dacplus.c"
Changed lines of the file:
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@@
+    (effects (font (size 1.27 1.27)) (justify left bottom))
+  )
+  (text "https://github.com/raspberrypi/linux/blob/rpi-5.15.y/sound/soc/bcm/hifiberry_dacplus.c"
+    (at 12.7 152.4 0)
     (effects (font (size 1.27 1.27)) (justify left bottom))
   )

Commit message: data5
Parts:
- C10, C8: footprint (none) -> Capacitor_SMD:C_0603_1608Metric_Pad1.08x0.95mm_HandSolder
- C11, C12, C14, C16, C17, C19, C2, C20, C23, C24, C3, C4, C5, C9: footprint (none) -> Capacitor_SMD:C_0402_1005Metric_Pad0.74x0.62mm_HandSolder
- C13, C15, C18, C22, C25, C6, C7: footprint (none) -> Capacitor_SMD:CP_Elec_4x5.4
- C21: value 10nH -> 1n; footprint (none) -> Capacitor_SMD:C_0805_2012Metric_Pad1.18x1.45mm_HandSolder
- C26: footprint (none) -> Capacitor_SMD:CP_Elec_5x5.4
- D2: footprint (none) -> LED_SMD:LED_0603_1608Metric_Pad1.05x0.95mm_HandSolder
- JP1, JP2, JP3, JP4: footprint (none) -> Jumper:SolderJumper-2_P1.3mm_Open_Pad1.0x1.5mm

Commit message: da
Parts:
- removed AE1: Antenna, Connector_PinHeader_2.54mm:PinHeader_1x01_P2.54mm_Vertical, symbol Device:Antenna
- removed AE2: Antenna_Loop, Connector_PinHeader_2.54mm:PinHeader_1x02_P2.54mm_Vertical, symbol Device:Antenna_Loop
- removed C1: 0.47u, Capacitor_SMD:C_1206_3216Metric_Pad1.33x1.80mm_HandSolder, symbol Device:C
- removed C2, C5: 0.1u, Capacitor_SMD:C_0402_1005Metric_Pad0.74x0.62mm_HandSolder, symbol Device:C
- removed C20: 33p, Capacitor_SMD:C_0402_1005Metric_Pad0.74x0.62mm_HandSolder, symbol Device:C
- removed C21: 1n, Capacitor_SMD:C_0805_2012Metric_Pad1.18x1.45mm_HandSolder, symbol Device:C
- removed L1: 4.7H, symbol Device:L
- removed L2: 100nH, symbol Device:L
- removed R4, R7, R8: 10k, symbol Device:R
- removed SW1: SW_SPDT, symbol Switch:SW_SPDT
- removed U2: Si4732, symbol locallib:Si4832
- removed U3: CM1213A-02, symbol locallib:CM1213A-02
Connections:
- no-connect marks 1 -> 0
