File: motorFullBridge.kicad_sch (KiCad schematic)
At the start: 22 parts

Commit message: data3543
Parts:
- added Q?: Q_NMOS_GSD, symbol Device:Q_NMOS_GSD
- added R? (x2): R, symbol Device:R
Connections:
- net EN is gone; now on net IN2: U?.7 (EN), U?.7 (EN)
- net +3V3: now also R?.2
- net GND: now also Q?.2 (S)
- net IN1: now also R?.1
- net IN2: now also Q?.3 (D), R?.1
- new net: Q?.1 (G), R?.2
Changed lines of the file:
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@@
   (junction (at 139.7 41.91) (diameter 0) (color 0 0 0 0)
+  )
+  (junction (at 110.49 107.95) (diameter 0) (color 0 0 0 0)
   )
   (junction (at 85.09 90.17) (diameter 0) (color 0 0 0 0)
@@
     (stroke (width 0) (type default) (color 0 0 0 0))
   )
+  (wire (pts (xy 35.56 110.49) (xy 40.64 110.49))
+    (stroke (width 0) (type default) (color 0 0 0 0))
+  )
   (wire (pts (xy 147.32 53.34) (xy 170.18 53.34))
     (stroke (width 0) (type default) (color 0 0 0 0))
@@
     (stroke (width 0) (type default) (color 0 0 0 0))
   )
+  (wire (pts (xy 25.4 105.41) (xy 30.48 105.41))
+    (stroke (width 0) (type default) (color 0 0 0 0))
+  )
   (wire (pts (xy 55.88 58.42) (xy 62.23 58.42))
     (stroke (width 0) (type default) (color 0 0 0 0))
@@
     (stroke (width 0) (type default) (color 0 0 0 0))
   )
+  (wire (pts (xy 110.49 107.95) (xy 118.11 107.95))
+    (stroke (width 0) (type default) (color 0 0 0 0))
+  )
   (wire (pts (xy 90.17 58.42) (xy 90.17 57.15))
     (stroke (width 0) (type default) (color 0 0 0 0))
@@
   )
   (wire (pts (xy 116.84 52.07) (xy 116.84 53.34))
+    (stroke (width 0) (type default) (color 0 0 0 0))
+  )
+  (wire (pts (xy 35.56 100.33) (xy 40.64 100.33))
     (stroke (width 0) (type default) (color 0 0 0 0))
   )
@@
     (effects (font (size 1.27 1.27)) (justify right bottom))
   )
+  (label "IN1" (at 95.25 113.03 180)
+    (effects (font (size 1.27 1.27)) (justify right bottom))
+  )
   (label "HO2" (at 162.56 46.99 0)
     (effects (font (size 1.27 1.27)) (justify left bottom))
@@
     (effects (font (size 1.27 1.27)) (justify right bottom))
   )
+  (label "EN" (at 86.36 107.95 0)
+    (effects (font (size 1.27 1.27)) (justify left bottom))
+  )
   (label "LO2" (at 162.56 59.69 0)
     (effects (font (size 1.27 1.27)) (justify left bottom))
@@
     (effects (font (size 1.27 1.27)) (justify right bottom))
   )
-  (label "IN2" (at 86.36 107.95 0)
+  (label "IN2" (at 118.11 107.95 0)
     (effects (font (size 1.27 1.27)) (justify left bottom))
   )
   (label "LO1" (at 101.6 59.69 180)
     (effects (font (size 1.27 1.27)) (justify right bottom))
+  )
+  (global_label "VDD" (shape passive) (at 35.56 100.33 180) (fields_autoplaced)
+    (effects (font (size 1.27 1.27)) (justify right))
+    (property "Intersheet References" "${INTERSHEET_REFS}" (id 0) (at 29.5183 100.2506 0)
+      (effects (font (size 1.27 1.27)) (justify right) hide)
+    )
+  )
+  (global_label "GND" (shape passive) (at 35.56 110.49 180) (fields_autoplaced)
+    (effects (font (size 1.27 1.27)) (justify right))
+    (property "Intersheet References" "${INTERSHEET_REFS}" (id 0) (at 29.2764 110.4106 0)
+      (effects (font (size 1.27 1.27)) (justify right) hide)
+    )
+  )
+  (global_label "BATT" (shape passive) (at 30.48 105.41 0) (fields_autoplaced)
+    (effects (font (size 1.27 1.27)) (justify left))
+    (property "Intersheet References" "${INTERSHEET_REFS}" (id 0) (at 37.1869 105.3306 0)
+      (effects (font (size 1.27 1.27)) (justify left) hide)
+    )
   )
   (hierarchical_label "IN1" (shape passive) (at 86.36 105.41 180)
@@
     (pin "2")
   )
+  (symbol (lib_id "power:GND") (at 40.64 110.49 0) (mirror y)
+    (in_bom yes) (on_board yes) (fields_autoplaced)
+    (property "Reference" "#PWR?" (id 0) (at 40.64 116.84 0)
+      (effects (font (size 1.27 1.27)) hide)
+    )
+    (property "Value" "GND" (id 1) (at 40.64 114.9334 0))
+    (property "Footprint" "" (id 2) (at 40.64 110.49 0)
+      (effects (font (size 1.27 1.27)) hide)
+    )
+    (property "Datasheet" "" (id 3) (at 40.64 110.49 0)
+      (effects (font (size 1.27 1.27)) hide)
+    )
+    (pin "1")
+  )
   (symbol (lib_id "power:GND") (at 33.02 62.23 0) (mirror y)
     (in_bom yes) (on_board yes) (fields_autoplaced)
@@
     (pin "1")
     (pin "2")
+  )
+  (symbol (lib_id "power:GND") (at 110.49 118.11 0) (mirror y)
+    (in_bom yes) (on_board yes) (fields_autoplaced)
+    (property "Reference" "#PWR?" (id 0) (at 110.49 124.46 0)
+      (effects (font (size 1.27 1.27)) hide)
+    )
+    (property "Value" "GND" (id 1) (at 110.49 122.5534 0))
+    (property "Footprint" "" (id 2) (at 110.49 118.11 0)
+      (effects (font (size 1.27 1.27)) hide)
+    )
+    (property "Datasheet" "" (id 3) (at 110.49 118.11 0)
+      (effects (font (size 1.27 1.27)) hide)
+    )
+    (pin "1")
+  )
+  (symbol (lib_id "power:+3V3") (at 40.64 100.33 0) (mirror y)
+    (in_bom yes) (on_board yes)
+    (property "Reference" "#PWR?" (id 0) (at 40.64 104.14 0)
+      (effects (font (size 1.27 1.27)) hide)
+    )
+    (property "Value" "+3V3" (id 1) (at 40.259 95.9358 0))
+    (property "Footprint" "" (id 2) (at 40.64 100.33 0)
+      (effects (font (size 1.27 1.27)) hide)
+    )
+    (property "Datasheet" "" (id 3) (at 40.64 100.33 0)
+      (effects (font (size 1.27 1.27)) hide)
+    )
+    (pin "1")
+  )
+  (symbol (lib_id "power:+3V3") (at 110.49 100.33 0) (mirror y)
+    (in_bom yes) (on_board yes)
+    (property "Reference" "#PWR?" (id 0) (at 110.49 104.14 0)
+      (effects (font (size 1.27 1.27)) hide)
+    )
+    (property "Value" "+3V3" (id 1) (at 110.109 95.9358 0))
+    (property "Footprint" "" (id 2) (at 110.49 100.33 0)
+      (effects (font (size 1.27 1.27)) hide)
+    )
+    (property "Datasheet" "" (id 3) (at 110.49 100.33 0)
+      (effects (font (size 1.27 1.27)) hide)
+    )
+    (pin "1")
   )
   (symbol (lib_id "power:+3V3") (at 85.09 60.96 0) (mirror y)
@@
     (pin "2")
   )
+  (symbol (lib_id "Device:Q_NMOS_GSD") (at 107.95 113.03 0)
+    (in_bom yes) (on_board yes) (fields_autoplaced)
+    (property "Reference" "Q?" (id 0) (at 113.157 112.1953 0)
+      (effects (font (size 1.27 1.27)) (justify left))
+    )
+    (property "Value" "Q_NMOS_GSD" (id 1) (at 113.157 114.7322 0)
+      (effects (font (size 1.27 1.27)) (justify left))
+    )
+    (property "Footprint" "" (id 2) (at 113.03 110.49 0)
+      (effects (font (size 1.27 1.27)) hide)
+    )
+    (property "Datasheet" "~" (id 3) (at 107.95 113.03 0)
+      (effects (font (size 1.27 1.27)) hide)
+    )
+    (pin "1")
+    (pin "2")
+    (pin "3")
+  )
   (symbol (lib_id "Device:R") (at 158.75 59.69 270) (mirror x)
     (in_bom yes) (on_board yes) (fields_autoplaced)
@@
     (pin "9")
   )
+  (symbol (lib_id "Device:R") (at 99.06 113.03 90)
+    (in_bom yes) (on_board yes) (fields_autoplaced)
+    (property "Reference" "R?" (id 0) (at 99.06 108.3142 90))
+    (property "Value" "R" (id 1) (at 99.06 110.8511 90))
+    (property "Footprint" "" (id 2) (at 99.06 114.808 90)
+      (effects (font (size 1.27 1.27)) hide)
+    )
+    (property "Datasheet" "~" (id 3) (at 99.06 113.03 0)
+      (effects (font (size 1.27 1.27)) hide)
+    )
+    (pin "1")
+    (pin "2")
+  )
   (symbol (lib_id "Device:D") (at 139.7 59.69 270)
     (in_bom yes) (on_board yes) (fields_autoplaced)
@@
       (effects (font (size 1.27 1.27)) hide)
     )
+    (pin "1")
+  )
+  (symbol (lib_id "Device:R") (at 110.49 104.14 180)
+    (in_bom yes) (on_board yes) (fields_autoplaced)
+    (property "Reference" "R?" (id 0) (at 112.268 103.3053 0)
+      (effects (font (size 1.27 1.27)) (justify right))
+    )
+    (property "Value" "R" (id 1) (at 112.268 105.8422 0)
+      (effects (font (size 1.27 1.27)) (justify right))
+    )
+    (property "Footprint" "" (id 2) (at 112.268 104.14 90)
+      (effects (font (size 1.27 1.27)) hide)
+    )
+    (property "Datasheet" "~" (id 3) (at 110.49 104.14 0)
+      (effects (font (size 1.27 1.27)) hide)
+    )
+    (pin "1")
+    (pin "2")
+  )
+  (symbol (lib_id "power:+BATT") (at 25.4 105.41 0)
+    (in_bom yes) (on_board yes) (fields_autoplaced)
+    (property "Reference" "#PWR?" (id 0) (at 25.4 109.22 0)
+      (effects (font (size 1.27 1.27)) hide)
+    )
+    (property "Value" "+BATT" (id 1) (at 25.4 101.8342 0))
+    (property "Footprint" "" (id 2) (at 25.4 105.41 0)
+      (effects (font (size 1.27 1.27)) hide)
+    )
+    (property "Datasheet" "" (id 3) (at 25.4 105.41 0)
+      (effects (font (size 1.27 1.27)) hide)
+    )
